File: PCB/Hackpad schematic.kicad_pcb (KiCad board)
At the start: 2 copper layers, 67 x 47 mm, 9 parts, among them SW1 SW_Push, SW2 SW_Push, SW3 SW_Push, SW4 SW_Push, SW5 RotaryEncoder_Switch, U1 MOUDLE-SEEEDUINO-XIAO

Commit message: Working LED Gerbers
Parts:
- D1, D2: footprint Care Package:SK6812MINI-E_fixed -> LED_SMD:LED_SK6812MINI-E_3.2x2.8mm_P1.5mm_ReverseMount
Connections:
- D1 pad 1: Net-(D1-DOUT) -> GND
- D1 pad 2: GND -> RGB_Lighting
- D1 pad 4: RGB_Lighting -> Net-(D1-DOUT)
- D2 pad 1: unconnected-(D2-DOUT-Pad1) -> GND
- D2 pad 2: GND -> Net-(D1-DOUT)
- D2 pad 4: Net-(D1-DOUT) -> unconnected-(D2-DOUT-Pad4)
Routing:
- net VCC: track 80.6 -> 53.4 mm
- net Net-(U1-PA5_A9_D9_MISO): track 62.2 -> 43.4 mm
- net RGB_Lighting: track 36.0 -> 48.6 mm, vias 0 -> 1
- net GND: track 122.0 -> 128.1 mm
- net Net-(D1-DOUT): track 22.2 -> 28.2 mm, vias 0 -> 2
- net Net-(U1-PA10_A2_D2): track 62.3 -> 66.4 mm
- net Net-(U1-PB09_A7_D7_RX): track 18.5 -> 15.2 mm
- net Net-(U1-PA4_A1_D1): track 63.6 -> 66.5 mm
- net Net-(U1-PA11_A3_D3): track 46.0 -> 48.8 mm
- net unconnected-(U1-PA9_A5_D5_SCL-Pad6): track 2.07 -> 0.00 mm
- net Net-(U1-PA7_A8_D8_SCK): track 17.9 -> 19.0 mm
- net Net-(U1-PA6_A10_D10_MOSI): track 20.3 -> 21.4 mm
- net unconnected-(U1-3V3-Pad12): track 1.04 -> 0.00 mm
- net unconnected-(U1-PB08_A6_D6_TX-Pad7): track 1.04 -> 0.00 mm
