File: PCB/Hackpad schematic.kicad_sch (KiCad schematic)
At the start: 7 parts, among them SW1 SW_Push, SW2 SW_Push, SW3 SW_Push, SW4 SW_Push, U1 MOUDLE-SEEEDUINO-XIAO

Commit message: Added rotary knob
Added rotary knob. Made skull smaller
Parts:
- added SW5: RotaryEncoder_Switch, Rotary_Encoder:RotaryEncoder_Alps_EC11E-Switch_Vertical_H20mm, symbol Device:RotaryEncoder_Switch
Connections:
- net GND: now also SW5.C, SW5.S1
- net at U1.2 (PA4_A1_D1): now also SW5.A
- net at U1.3 (PA10_A2_D2): now also SW5.B
- net at U1.4 (PA11_A3_D3): now also SW5.S2

Commit message: Working LED Gerbers
Parts:
- D1, D2: footprint Care Package:SK6812MINI-E_fixed -> LED_SMD:LED_SK6812MINI-E_3.2x2.8mm_P1.5mm_ReverseMount; symbol LED:NeoPixel_THT -> LED:SK6812MINI-E
Connections:
- net GND: now also D1.1 (VSS), D2.1 (VSS); no longer D1.2 (GND), D2.2 (GND)
- net RGB_Lighting: now also D1.2 (DIN); no longer D1.4 (DIN)
- net at D2.4 (DOUT): no longer D1.1 (DOUT)
- new net: D1.4 (DOUT), D2.2 (DIN)
Changed lines of the file:
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@@
 	)
 	(symbol
-		(lib_id "LED:NeoPixel_THT")
+		(lib_id "LED:SK6812MINI-E")
 		(at 69.85 91.44 0)
 		(unit 1)
@@
 			)
 		)
-		(property "Footprint" "Care Package:SK6812MINI-E_fixed"
+		(property "Footprint" "LED_SMD:LED_SK6812MINI-E_3.2x2.8mm_P1.5mm_ReverseMount"
 			(at 71.12 99.06 0)
 			(hide yes)
@@
 			)
 		)
-		(property "Datasheet" "https://www.adafruit.com/product/1938"
+		(property "Datasheet" "https://www.lcsc.com/datasheet/C5149201.pdf"
 			(at 72.39 100.965 0)
 			(hide yes)
@@
 			)
 		)
-		(property "Description" "RGB LED with integrated controller, 5mm/8mm LED package"
+		(property "Description" "RGB LED with integrated controller"
 			(at 69.85 91.44 0)
 			(hide yes)
@@
 	)
 	(symbol
-		(lib_id "LED:NeoPixel_THT")
+		(lib_id "LED:SK6812MINI-E")
 		(at 43.18 91.44 0)
 		(unit 1)
@@
 		(fields_autoplaced yes)
 		(property "Reference" "D1"
-			(at 55.88 85.0198 0)
+			(at 30.48 85.0198 0)
 			(show_name no)
 			(do_not_autoplace no)
@@
 		)
 		(property "Value" "NeoPixel_THT"
-			(at 55.88 87.5598 0)
-			(show_name no)
-			(do_not_autoplace no)
-			(effects
-				(font
-					(size 1.27 1.27)
-				)
-			)
-		)
-		(property "Footprint" "Care Package:SK6812MINI-E_fixed"
+			(at 30.48 87.5598 0)
+			(show_name no)
+			(do_not_autoplace no)
+			(effects
+				(font
+					(size 1.27 1.27)
+				)
+			)
+		)
+		(property "Footprint" "LED_SMD:LED_SK6812MINI-E_3.2x2.8mm_P1.5mm_ReverseMount"
 			(at 44.45 99.06 0)
 			(hide yes)
@@
 			)
 		)
-		(property "Datasheet" "https://www.adafruit.com/product/1938"
+		(property "Datasheet" "https://www.lcsc.com/datasheet/C5149201.pdf"
 			(at 45.72 100.965 0)
 			(hide yes)
@@
 			)
 		)
-		(property "Description" "RGB LED with integrated controller, 5mm/8mm LED package"
+		(property "Description" "RGB LED with integrated controller"
 			(at 43.18 91.44 0)
 			(hide yes)
