File: PCB/GD-Hackpad/Hackpad schematic.kicad_pcb (KiCad board)
At the start: 2 copper layers, 67 x 47 mm, 9 parts, among them SW1 SW_Push, SW2 SW_Push, SW3 SW_Push, SW4 SW_Push, SW5 RotaryEncoder_Switch, U1 MOUDLE-SEEEDUINO-XIAO

Commit message: Separate kicad files for LED version
Parts:
- D1, D2: footprint LED_SMD:LED_SK6812MINI-E_3.2x2.8mm_P1.5mm_ReverseMount -> Care Package:SK6812MINI-E_fixed
Connections:
- D1 pad 1: GND -> Net-(D1-DOUT)
- D1 pad 2: RGB_Lighting -> GND
- D1 pad 4: Net-(D1-DOUT) -> RGB_Lighting
- D2 pad 1: GND -> unconnected-(D2-DOUT-Pad1)
- D2 pad 2: Net-(D1-DOUT) -> GND
- D2 pad 4: unconnected-(D2-DOUT-Pad4) -> Net-(D1-DOUT)
Routing:
- net VCC: track 53.4 -> 80.6 mm
- net Net-(U1-PA5_A9_D9_MISO): track 43.4 -> 62.2 mm
- net RGB_Lighting: track 48.6 -> 36.0 mm, vias 1 -> 0
- net GND: track 128.1 -> 122.0 mm
- net Net-(D1-DOUT): track 28.2 -> 22.2 mm, vias 2 -> 0
- net Net-(U1-PA10_A2_D2): track 66.4 -> 62.3 mm
- net Net-(U1-PB09_A7_D7_RX): track 15.2 -> 18.5 mm
- net Net-(U1-PA4_A1_D1): track 66.5 -> 63.6 mm
- net Net-(U1-PA11_A3_D3): track 48.8 -> 46.0 mm
- net unconnected-(U1-PA9_A5_D5_SCL-Pad6): track 0.00 -> 2.07 mm
- net Net-(U1-PA7_A8_D8_SCK): track 19.0 -> 17.9 mm
- net Net-(U1-PA6_A10_D10_MOSI): track 21.4 -> 20.3 mm
- net unconnected-(U1-3V3-Pad12): track 0.00 -> 1.04 mm
- net unconnected-(U1-PB08_A6_D6_TX-Pad7): track 0.00 -> 1.04 mm
