File: PCB/GD-Hackpad/Hackpad schematic.kicad_sch (KiCad schematic)
At the start: 8 parts, among them SW1 SW_Push, SW2 SW_Push, SW3 SW_Push, SW4 SW_Push, SW5 RotaryEncoder_Switch, U1 MOUDLE-SEEEDUINO-XIAO

Commit message: Separate kicad files for LED version
Parts:
- D1, D2: footprint LED_SMD:LED_SK6812MINI-E_3.2x2.8mm_P1.5mm_ReverseMount -> Care Package:SK6812MINI-E_fixed; symbol LED:SK6812MINI-E -> LED:NeoPixel_THT
Connections:
- net GND: now also D1.2 (GND), D2.2 (GND); no longer D1.1 (VSS), D2.1 (VSS)
- net RGB_Lighting: now also D1.4 (DIN); no longer D1.2 (DIN)
- net at D2.4 (DIN): now also D1.1 (DOUT)
Changed lines of the file:
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@@
 	)
 	(symbol
-		(lib_id "LED:SK6812MINI-E")
+		(lib_id "LED:NeoPixel_THT")
 		(at 69.85 91.44 0)
 		(unit 1)
@@
 			)
 		)
-		(property "Footprint" "LED_SMD:LED_SK6812MINI-E_3.2x2.8mm_P1.5mm_ReverseMount"
+		(property "Footprint" "Care Package:SK6812MINI-E_fixed"
 			(at 71.12 99.06 0)
 			(hide yes)
@@
 			)
 		)
-		(property "Datasheet" "https://www.lcsc.com/datasheet/C5149201.pdf"
+		(property "Datasheet" "https://www.adafruit.com/product/1938"
 			(at 72.39 100.965 0)
 			(hide yes)
@@
 			)
 		)
-		(property "Description" "RGB LED with integrated controller"
+		(property "Description" "RGB LED with integrated controller, 5mm/8mm LED package"
 			(at 69.85 91.44 0)
 			(hide yes)
@@
 	)
 	(symbol
-		(lib_id "LED:SK6812MINI-E")
+		(lib_id "LED:NeoPixel_THT")
 		(at 43.18 91.44 0)
 		(unit 1)
@@
 		(fields_autoplaced yes)
 		(property "Reference" "D1"
-			(at 30.48 85.0198 0)
+			(at 55.88 85.0198 0)
 			(show_name no)
 			(do_not_autoplace no)
@@
 		)
 		(property "Value" "NeoPixel_THT"
-			(at 30.48 87.5598 0)
-			(show_name no)
-			(do_not_autoplace no)
-			(effects
-				(font
-					(size 1.27 1.27)
-				)
-			)
-		)
-		(property "Footprint" "LED_SMD:LED_SK6812MINI-E_3.2x2.8mm_P1.5mm_ReverseMount"
+			(at 55.88 87.5598 0)
+			(show_name no)
+			(do_not_autoplace no)
+			(effects
+				(font
+					(size 1.27 1.27)
+				)
+			)
+		)
+		(property "Footprint" "Care Package:SK6812MINI-E_fixed"
 			(at 44.45 99.06 0)
 			(hide yes)
@@
 			)
 		)
-		(property "Datasheet" "https://www.lcsc.com/datasheet/C5149201.pdf"
+		(property "Datasheet" "https://www.adafruit.com/product/1938"
 			(at 45.72 100.965 0)
 			(hide yes)
@@
 			)
 		)
-		(property "Description" "RGB LED with integrated controller"
+		(property "Description" "RGB LED with integrated controller, 5mm/8mm LED package"
 			(at 43.18 91.44 0)
 			(hide yes)
